Commit message: added no wheel version

File: resources/robots/wheely/URDFs/V2-8.urdf (robot description, URDF)
Before this commit: robot wheely, 18 links, 17 joints
Links:
- removed link trunk
- link base: mass None -> 1.0520000000000000462; geometry collision mesh filename=../meshes/V2.8/trunk.stl; visual mesh filename=../meshes/V2.8/trunk.stl
Joints:
- removed joint floating_base
- joint BLHU: parent trunk -> base
- joint BRHU: parent trunk -> base
- joint FLHU: parent trunk -> base
- joint FRHU: parent trunk -> base
