Commit message: New Goal Oriented Training; New Training System; New Mixture of Experts Selector Algorithm; tldr, new everything

File: resources/robots/wheely/URDFs/V2-9.urdf (robot description, URDF)
Before this commit: robot wheely, 17 links, 16 joints
Joints:
- joint BLW: type revolute -> continuous
- joint BRW: type revolute -> continuous
- joint FLW: type revolute -> continuous
- joint FRW: type revolute -> continuous
