Commit message: Working motors, modified rewards - now walking

File: resources/robots/anymal_c/urdf/anymal_c.urdf (robot description, URDF)
Before this commit: robot anymal, 77 links, 76 joints
Links:
- removed link 
- added link LF_HAA, mass 2.04; visual mesh filename=../meshes/drive.dae scale=1.0 1.0 1.0
